Commit message: vel scaling factor works but not accel

File: ur_description/urdf/ur3_joint_limited_robot.urdf.xacro (robot description, xacro)
@@ -8,19 +8,4 @@
   <!-- arm -->
   <xacro:ur3_robot prefix="" joint_limited="true"/>
-	<link name="${prefix}spindle">
-	    <visual>
-	   	     <geometry>
-	          <mesh filename="package://ur_description/meshes/ur3/visual/spindle.stl"/>
-	        </geometry>
-	        <material name="LightGrey">
-	          <color rgba="0.7 0.7 0.7 1.0"/>
-	        </material>
-	  	</visual>
-	  	<collision>
-	        <geometry>
-	          <mesh filename="package://ur_description/meshes/ur3/visual/spindle.stl"/>
-	        </geometry>
-	  	</collision>
-	</link>
   <link name="world" />
   <joint name="world_joint" type="fixed">
