Commit message: added spindle

File: ur_description/urdf/ur3.urdf.xacro (robot description, xacro)
@@ -269,4 +269,24 @@
       </collision>
     </link>
+    <link name="${prefix}spindle">
+        <visual>
+	   	     <geometry>
+	          <mesh filename="package://ur_description/meshes/ur3/visual/spindle.stl"/>
+	        </geometry>
+	        <material name="LightGrey">
+	          <color rgba="0.7 0.7 0.7 1.0"/>
+	        </material>
+      	</visual>
+      	<collision>
+	        <geometry>
+	          <mesh filename="package://ur_description/meshes/ur3/visual/spindle.stl"/>
+	        </geometry>
+      	</collision>
+  	</link>
+    <joint name="${prefix}spindle" type="fixed">
+	      <origin xyz="0 0 0" rpy="0 0 0"/>
+	      <parent link="${prefix}tool0"/>
+	      <child link="${prefix}spindle"/>
+	</joint>
     <xacro:ur_arm_transmission prefix="${prefix}" />
     <xacro:ur_arm_gazebo prefix="${prefix}" />

File: ur_description/urdf/ur3_joint_limited_robot.urdf.xacro (robot description, xacro)
@@ -8,4 +8,19 @@
   <!-- arm -->
   <xacro:ur3_robot prefix="" joint_limited="true"/>
+	<link name="${prefix}spindle">
+	    <visual>
+	   	     <geometry>
+	          <mesh filename="package://ur_description/meshes/ur3/visual/spindle.stl"/>
+	        </geometry>
+	        <material name="LightGrey">
+	          <color rgba="0.7 0.7 0.7 1.0"/>
+	        </material>
+	  	</visual>
+	  	<collision>
+	        <geometry>
+	          <mesh filename="package://ur_description/meshes/ur3/visual/spindle.stl"/>
+	        </geometry>
+	  	</collision>
+	</link>
   <link name="world" />
   <joint name="world_joint" type="fixed">

Commit message: added surface

File: ur_description/urdf/ur3.urdf.xacro (robot description, xacro)
@@ -52,4 +52,22 @@
   </xacro:macro>
   <xacro:macro name="ur3_robot" params="prefix joint_limited">
+    <joint name="${prefix}base_plate" type="fixed">
+      <parent link="${prefix}base_link" />
+      <child link = "${prefix}base_plate_link" />
+      <origin xyz="0 0 0" rpy="0 0 0" />
+    </joint>
+    <link name="${prefix}base_plate_link">
+     <visual>
+        <geometry>
+          <box size="1.0 1.0 0.01"/>
+        </geometry>
+      </visual>
+      <collision>
+        <geometry>
+          <box size="1.0 1.0 0.01"/>
+        </geometry>
+      </collision>
+    <origin rpy="0 0 0" xyz="0 0 -0.05"/>
+    </link>
     <link name="${prefix}base_link" >
       <visual>

Commit message: added box

File: ur_description/urdf/ur3.urdf.xacro (robot description, xacro)
@@ -306,4 +306,24 @@
 	      <parent link="${prefix}tool0"/>
 	      <child link="${prefix}spindle"/>
+	  </joint>
+    <link name="${prefix}box_link">
+        <visual>
+	   	     <geometry>
+	          <mesh filename="package://ur_description/meshes/ur3/visual/box.stl"/>
+	        </geometry>
+	        <material name="LightGrey">
+	          <color rgba="0.7 0.7 0.7 1.0"/>
+	        </material>
+      	</visual>
+      	<collision>
+	        <geometry>
+	          <mesh filename="package://ur_description/meshes/ur3/visual/box.stl"/>
+	        </geometry>
+      	</collision>
+  	</link>
+    <joint name="${prefix}box_joint" type="fixed">
+	      <origin xyz="0 0 0" rpy="0 0 0"/>
+	      <parent link="${prefix}world"/>
+	      <child link="${prefix}box_link"/>
 	</joint>
     <xacro:ur_arm_transmission prefix="${prefix}" />

Commit message: new spidle

File: ur_description/urdf/ur3.urdf.xacro (robot description, xacro)
@@ -303,5 +303,5 @@
   	</link>
     <joint name="${prefix}spindle" type="fixed">
-	      <origin xyz="0 0 0" rpy="0 0 0"/>
+	      <origin xyz="0 0 0.1" rpy="0 0 0"/>
 	      <parent link="${prefix}tool0"/>
 	      <child link="${prefix}spindle"/>

Commit message: minor

File: ur_description/urdf/ur3.urdf.xacro (robot description, xacro)
@@ -303,5 +303,5 @@
   	</link>
     <joint name="${prefix}spindle" type="fixed">
-	      <origin xyz="0 0 0.1" rpy="0 0 0"/>
+	      <origin xyz="0 0 0" rpy="0 0 0"/>
 	      <parent link="${prefix}tool0"/>
 	      <child link="${prefix}spindle"/>

Commit message: init

File: ur_description/urdf/ur3.urdf.xacro (robot description, xacro)
@@ -52,22 +52,4 @@
   </xacro:macro>
   <xacro:macro name="ur3_robot" params="prefix joint_limited">
-    <joint name="${prefix}base_plate" type="fixed">
-      <parent link="${prefix}base_link" />
-      <child link = "${prefix}base_plate_link" />
-      <origin xyz="0 0 0" rpy="0 0 0" />
-    </joint>
-    <link name="${prefix}base_plate_link">
-     <visual>
-        <geometry>
-          <box size="1.0 1.0 0.01"/>
-        </geometry>
-      </visual>
-      <collision>
-        <geometry>
-          <box size="1.0 1.0 0.01"/>
-        </geometry>
-      </collision>
-    <origin rpy="0 0 0" xyz="0 0 -0.05"/>
-    </link>
     <link name="${prefix}base_link" >
       <visual>

Commit message: refined

File: ur_description/urdf/ur3.urdf.xacro (robot description, xacro)
@@ -107,5 +107,5 @@
       <axis xyz="0 1 0" />
       <xacro:unless value="${joint_limited}">
-        <limit lower="${-2.0 * pi}" upper="${2.0 * pi}" effort="330.0" velocity="2.16"/>
+        <limit lower="${-2.2 * pi}" upper="${2.2 * pi}" effort="330.0" velocity="2.16"/>
       </xacro:unless>
       <xacro:if value="${joint_limited}">
@@ -234,5 +234,5 @@
       </xacro:unless>
       <xacro:if value="${joint_limited}">
-        <limit lower="${-pi}" upper="${pi}" effort="54.0" velocity="3.2"/>
+        <limit lower="${-2.0* pi}" upper="${2.0*pi}" effort="54.0" velocity="3.2"/>
       </xacro:if>
       <dynamics damping="0.0" friction="0.0"/>

Commit message: new box

File: ur_description/urdf/ur3.urdf.xacro (robot description, xacro)
@@ -73,5 +73,5 @@
       <parent link="${prefix}base_link" />
       <child link = "${prefix}shoulder_link" />
-      <origin xyz="0.0 0.0 ${shoulder_height}" rpy="0.0 0.0 0.0" />
+      <origin xyz="0.0 0.0 ${shoulder_height}" rpy="0.0 0.0 1.57" />
       <axis xyz="0 0 1" />
       <xacro:unless value="${joint_limited}">

Commit message: box updated

File: ur_description/urdf/ur3.urdf.xacro (robot description, xacro)
@@ -261,4 +261,23 @@
       <origin xyz="0.0 ${wrist_3_length} 0.0" rpy="0.0 0.0 ${pi/2.0}" />
     </joint>
+    <link name="${prefix}front_link">
+      <!-- <visual>
+        <geometry>
+          <box size="0.01 0.01 0.01"/>
+        </geometry>
+        <origin rpy="0 0 0" xyz="-0.01 0 0"/>
+      </visual> -->
+      <collision>
+        <geometry>
+          <box size="0.8 0.01 0.7"/>
+        </geometry>
+        <origin rpy="0 0 0" xyz="-0.23 0.25 0.35"/>
+      </collision>
+    </link>
+    <joint name="${prefix}front_panel_joint" type="fixed">
+      <parent link="${prefix}world" />
+      <child link = "${prefix}front_link" />
+      <origin xyz="0.0 0.0 0.0" rpy="0.0 0.0 0.0" />
+    </joint>
     <link name="${prefix}ee_link">
       <collision>

File: ur_description/urdf/ur3_joint_limited_robot.urdf.xacro (robot description, xacro)
@@ -23,5 +23,5 @@
     <parent link="world" />
     <child link = "base_link" />
-    <origin xyz="0.0 0.0 0.0" rpy="0.0 0.0 0.0" />
+    <origin xyz="0.0 0.0 0.038" rpy="0.0 0.0 0.0" />
   </joint>
 </robot>

Commit message: minor

File: ur_description/urdf/ur3.urdf.xacro (robot description, xacro)
@@ -304,5 +304,5 @@
   	</link>
     <joint name="${prefix}spindle" type="fixed">
-	      <origin xyz="0 0 0" rpy="0 0 0"/>
+	      <origin xyz="0 0 0" rpy="0 0 3.14"/>
 	      <parent link="${prefix}tool0"/>
 	      <child link="${prefix}spindle"/>

File: ur_description/urdf/ur3_robot.urdf.xacro (robot description, xacro)
@@ -23,5 +23,5 @@
     <parent link="world" />
     <child link = "base_link" />
-    <origin xyz="0.0 0.0 0.0" rpy="0.0 0.0 0.0" />
+    <origin xyz="0.0 0.0 0.038" rpy="0.0 0.0 0.0" />
   </joint>
 </robot>
